File: 12-5_Convertor/12-5Convertor.brd (EAGLE design)
At the start: 29.1 x 41.3 mm, 14 parts, among them IC1 ACS764, U1 LM2678

Commit message: rip up wires
Routing:
- net +5V: track 52.4 -> 0.00 mm, vias 2 -> 0
- net GND: track 10.5 -> 0.00 mm, vias 11 -> 0
- net N$2: track 6.58 -> 0.00 mm
- net +3V3: track 2.08 -> 0.00 mm
- removed copper zone on layer 1, net +12V
- removed copper zone on layer 1, net +5V
- removed copper zone on layer 16, net GND
- removed copper zone on layer 1, net N$3
Other:
- board size 29.1 x 41.3 mm -> 67.2 x 59 mm
- board text removed: "+12V"
- board text removed: "5V"
- board text removed: "Designed by Luke McBee, Richard Shen, Jeff Geiss, and Dimcho Karakashev +12V to +5V Buck Regulator 11/8/2015"
- board text removed: "GND"
- board text removed: "ON/OFF"

Commit message: why I need to commit?
Parts:
- moved U$3 53.6 mm to (38.4, 62.2), turned to 90 degrees
Changed lines of the file:
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@@
 <attribute name="NAME" x="33.186" y="30.87" size="1.27" layer="21"/>
 </element>
-<element name="U$3" library="PowerComponents" package="NCP1117" value="NCP1117" x="26.67" y="9.906"/>
+<element name="U$3" library="PowerComponents" package="NCP1117" value="NCP1117" x="38.354" y="62.23" rot="R90"/>
 <element name="C7" library="SparkFun-Passives" package="0603-CAP" value="10UF" x="21.336" y="4.064"/>
 <element name="C8" library="SparkFun-Passives" package="0603-CAP" value="10UF" x="21.336" y="1.524"/>
@@
 <wire x1="43.18" y1="24.5" x2="46.2788" y2="24.13" width="0" layer="19" extent="1-1"/>
 <wire x1="37.592" y1="22.658" x2="43.18" y2="24.5" width="0" layer="19" extent="1-1"/>
-<wire x1="24.37" y1="6.756" x2="37.592" y2="22.658" width="0" layer="19" extent="1-1"/>
-<wire x1="22.186" y1="4.064" x2="24.37" y2="6.756" width="0" layer="19" extent="1-1"/>
+<wire x1="41.504" y1="59.93" x2="37.592" y2="22.658" width="0" layer="19" extent="1-1"/>
+<wire x1="22.186" y1="4.064" x2="41.504" y2="59.93" width="0" layer="19" extent="1-1"/>
 <wire x1="22.186" y1="1.524" x2="22.186" y2="4.064" width="0" layer="19" extent="1-1"/>
 <wire x1="18.08" y1="-1.708" x2="22.186" y2="1.524" width="0" layer="19" extent="1-1"/>
@@
 <wire x1="43.18" y1="26.3" x2="46.2788" y2="26.67" width="0" layer="19" extent="1-1"/>
 <wire x1="37.592" y1="29.158" x2="43.18" y2="26.3" width="0" layer="19" extent="1-1"/>
-<wire x1="28.97" y1="6.756" x2="37.592" y2="29.158" width="0" layer="19" extent="1-1"/>
-<wire x1="20.486" y1="4.064" x2="28.97" y2="6.756" width="0" layer="19" extent="1-1"/>
+<wire x1="41.504" y1="64.53" x2="37.592" y2="29.158" width="0" layer="19" extent="1-1"/>
+<wire x1="20.486" y1="4.064" x2="41.504" y2="64.53" width="0" layer="19" extent="1-1"/>
 </signal>
 <signal name="+5V">
@@
 <contactref element="U$3" pad="OUT"/>
 <contactref element="C8" pad="1"/>
-<wire x1="20.486" y1="1.524" x2="26.67" y2="6.756" width="0" layer="19" extent="1-1"/>
+<wire x1="20.486" y1="1.524" x2="41.504" y2="62.23" width="0" layer="19" extent="1-1"/>
 <wire x1="20.486" y1="-2.54" x2="20.486" y2="1.524" width="0" layer="19" extent="1-1"/>
 </signal>
